File: wireless_measurement_ard.sch (KiCad schematic (older format))
At the start: 25 parts, among them J1 Conn_01x08, SW1 SW_SPDT, U1 EFM8LB1, U2 JDY-08, U3 MCP16415, U4 MAX9938, U5 MAX9938, U6 EFM8LB1x-QFP32

Commit message: Halved the size of the board
Parts:
- removed EFM8_Prog1: Conn_01x03, Connector_PinHeader_2.54mm:PinHeader_1x03_P2.54mm_Vertical, symbol Connector_Generic:Conn_01x03
- removed U6: EFM8LB1x-QFP32, Package_QFP:LQFP-32_7x7mm_P0.8mm, symbol wireless_measurement_ard-rescue:EFM8LB1x-QFP32-gen_lib
- added J2: Tag-Connect, Connector:Tag-Connect_TC2030-IDC-NL_2x03_P1.27mm_Vertical, symbol Connector_Generic:Conn_02x03_Odd_Even
- added R6: 1k, Resistor_SMD:R_0603_1608Metric_Pad0.98x0.95mm_HandSolder, symbol Device:R
- renumbered R2 to R1, R1 to R2
Connections:
- net +3V3: now also J1.7 (Pin_7), R6.1
- net A3: now also J1.6 (Pin_6); no longer J1.7 (Pin_7)
- net BATT: now also J2.1 (Pin_1)
- net C1_IN: now also J1.2 (Pin_2); no longer J1.1 (Pin_1)
- net C1_OUT: now also J1.1 (Pin_1); no longer J1.2 (Pin_2)
- net C2CK: now also J2.3 (Pin_3), R6.2
- net C2D: now also J2.5 (Pin_5)
- net C2_IN: now also J1.4 (Pin_4); no longer J1.3 (Pin_3)
- net C2_OUT: now also J1.3 (Pin_3); no longer J1.4 (Pin_4)
- net GND: now also J2.6 (Pin_6); no longer J1.6 (Pin_6)
Changed lines of the file:
@@
 	9250 2100 9450 2100
 $Comp
-L Device:R R1
+L Device:R R2
 U 1 1 60F771F1
 P 9450 2250
-F 0 "R1" H 9520 2296 50  0000 L CNN
+F 0 "R2" H 9520 2296 50  0000 L CNN
 F 1 "5R3" H 9520 2205 50  0000 L CNN
 F 2 "Resistor_SMD:R_0805_2012Metric_Pad1.15x1.40mm_HandSolder" V 9380 2250 50  0001 C CNN
@@
 	9350 1550 9450 1550
 $Comp
-L Device:R R2
+L Device:R R1
 U 1 1 60F77736
 P 9450 1700
-F 0 "R2" H 9520 1746 50  0000 L CNN
+F 0 "R1" H 9520 1746 50  0000 L CNN
 F 1 "5R3" H 9520 1655 50  0000 L CNN
 F 2 "Resistor_SMD:R_0805_2012Metric_Pad1.15x1.40mm_HandSolder" V 9380 1700 50  0001 C CNN
@@
 	1    0    0    -1
 $EndComp
-Text GLabel 9300 3400 0    50   Input ~ 0
+Text GLabel 9300 3300 0    50   Input ~ 0
 A3
 Text GLabel 9300 3200 0    50   Input ~ 0
@@
 L power:GND #PWR0106
 U 1 1 60F9306D
-P 9150 3500
-F 0 "#PWR0106" H 9150 3250 50  0001 C CNN
-F 1 "GND" H 9155 3327 50  0000 C CNN
-F 2 "" H 9150 3500 50  0001 C CNN
-F 3 "" H 9150 3500 50  0001 C CNN
-	1    9150 3500
+P 9100 3500
+F 0 "#PWR0106" H 9100 3250 50  0001 C CNN
+F 1 "GND" V 9100 3300 50  0000 C CNN
+F 2 "" H 9100 3500 50  0001 C CNN
+F 3 "" H 9100 3500 50  0001 C CNN
+	1    9100 3500
 	0    1    1    0
 $EndComp
-$Comp
-L power:GND #PWR0105
-U 1 1 60F92C2D
-P 9150 3300
-F 0 "#PWR0105" H 9150 3050 50  0001 C CNN
-F 1 "GND" H 9155 3127 50  0000 C CNN
-F 2 "" H 9150 3300 50  0001 C CNN
-F 3 "" H 9150 3300 50  0001 C CNN
-	1    9150 3300
-	0    1    1    0
-$EndComp
-Wire Wire Line
-	9150 3300 9300 3300
-Wire Wire Line
-	9150 3500 9300 3500
 Text GLabel 9800 1650 2    50   Input ~ 0
 C1_IN
@@
 Wire Wire Line
 	9650 1650 9800 1650
-Text GLabel 9300 2800 0    50   Input ~ 0
+Text GLabel 9300 2900 0    50   Input ~ 0
 C1_IN
 Text GLabel 9800 1750 2    50   Input ~ 0
 C1_OUT
-Text GLabel 9300 2900 0    50   Input ~ 0
+Text GLabel 9300 2800 0    50   Input ~ 0
 C1_OUT
+Text GLabel 9300 3100 0    50   Input ~ 0
+C2_IN
 Text GLabel 9300 3000 0    50   Input ~ 0
-C2_IN
-Text GLabel 9300 3100 0    50   Input ~ 0
 C2_OUT
 Text GLabel 8550 4250 0    50   Input ~ 0
@@
 	8550 2300 8550 2400
 Connection ~ 8550 2400
-Text GLabel 3650 5500 2    50   Input ~ 0
-A0
-Text GLabel 3650 5400 2    50   Input ~ 0
-A1
-Text GLabel 3650 5300 2    50   Input ~ 0
-A2
-Text GLabel 3650 5200 2    50   Input ~ 0
-A3
 $Comp
 L power:+3.3V #PWR0118
@@
 $EndComp
 $Comp
-L wireless_measurement_ard-rescue:EFM8LB1x-QFP32-gen_lib U6
-U 1 1 6100BE6A
-P 3150 4900
-F 0 "U6" H 3150 5965 50  0000 C CNN
-F 1 "EFM8LB1x-QFP32" H 3150 5874 50  0000 C CNN
-F 2 "Package_QFP:LQFP-32_7x7mm_P0.8mm" H 3150 4650 50  0001 C CNN
-F 3 "" H 3150 4650 50  0001 C CNN
-	1    3150 4900
-	1    0    0    -1
-$EndComp
-Wire Wire Line
-	2650 4400 2200 4400
-Text GLabel 2650 4500 0    50   Input ~ 0
-C2CK
-Text GLabel 2650 4600 0    50   Input ~ 0
-C2D
-$Comp
 L Device:C C6
 U 1 1 610112E3
@@
 	1    0    0    -1
 $EndComp
-Connection ~ 2200 4400
 $Comp
 L Device:C C5
@@
 Wire Wire Line
 	2200 4400 1950 4400
-Wire Wire Line
-	1950 4300 2650 4300
 $Comp
 L power:GND #PWR0119
@@
 Wire Wire Line
 	2100 4700 2200 4700
-Text GLabel 3650 4500 2    50   Input ~ 0
-ARD_RX
-Text GLabel 3650 4400 2    50   Input ~ 0
-ARD_TX
-$Comp
-L power:GND #PWR0120
-U 1 1 61018C99
-P 2650 4200
-F 0 "#PWR0120" H 2650 3950 50  0001 C CNN
-F 1 "GND" H 2655 4027 50  0000 C CNN
-F 2 "" H 2650 4200 50  0001 C CNN
-F 3 "" H 2650 4200 50  0001 C CNN
-	1    2650 4200
-	0    1    1    0
-$EndComp
 Text GLabel 3850 1300 2    50   Input ~ 0
 STATUS
-Text GLabel 3650 5100 2    50   Input ~ 0
-STATUS
-Connection ~ 1950 4300
 Connection ~ 1950 4400
-$Comp
-L Connector_Generic:Conn_01x03 EFM8_Prog1
-U 1 1 61023B63
-P 7650 3400
-F 0 "EFM8_Prog1" H 7730 3442 50  0000 L CNN
-F 1 "Conn_01x03" H 7730 3351 50  0000 L CNN
-F 2 "Connector_PinHeader_2.54mm:PinHeader_1x03_P2.54mm_Vertical" H 7650 3400 50  0001 C CNN
-F 3 "~" H 7650 3400 50  0001 C CNN
-	1    7650 3400
-	1    0    0    -1
-$EndComp
 $Comp
 L power:GND #PWR0121
 U 1 1 610243BD
-P 7450 3500
-F 0 "#PWR0121" H 7450 3250 50  0001 C CNN
-F 1 "GND" H 7455 3327 50  0000 C CNN
-F 2 "" H 7450 3500 50  0001 C CNN
-F 3 "" H 7450 3500 50  0001 C CNN
-	1    7450 3500
-	1    0    0    -1
-$EndComp
-Text GLabel 7450 3400 0    50   Input ~ 0
+P 5350 3600
+F 0 "#PWR0121" H 5350 3350 50  0001 C CNN
+F 1 "GND" H 5355 3427 50  0000 C CNN
+F 2 "" H 5350 3600 50  0001 C CNN
+F 3 "" H 5350 3600 50  0001 C CNN
+	1    5350 3600
+	1    0    0    -1
+$EndComp
+Text GLabel 4850 3600 0    50   Input ~ 0
 C2D
-Text GLabel 7450 3300 0    50   Input ~ 0
+Text GLabel 4850 3500 0    50   Input ~ 0
 C2CK
 Wire Wire Line
 	8550 4450 8950 4450
-Text GLabel 3650 5000 2    50   Input ~ 0
-PWRC
 $Comp
 L Switch:SW_SPDT SW1
@@
 L power:+3.3V #PWR0109
 U 1 1 611EE56A
-P 4500 5250
-F 0 "#PWR0109" H 4500 5100 50  0001 C CNN
-F 1 "+3.3V" H 4515 5423 50  0000 C CNN
-F 2 "" H 4500 5250 50  0001 C CNN
-F 3 "" H 4500 5250 50  0001 C CNN
-	1    4500 5250
-	0    -1   -1   0
-$EndComp
-$Comp
-L power:+3.3V #PWR0110
-U 1 1 611EF11F
-P 4500 5350
-F 0 "#PWR0110" H 4500 5200 50  0001 C CNN
-F 1 "+3.3V" H 4515 5523 50  0000 C CNN
-F 2 "" H 4500 5350 50  0001 C CNN
-F 3 "" H 4500 5350 50  0001 C CNN
-	1    4500 5350
-	0    -1   -1   0
-$EndComp
-Text GLabel 4500 5450 0    50   Input ~ 0
+P 4150 5150
+F 0 "#PWR0109" H 4150 5000 50  0001 C CNN
+F 1 "+3.3V" H 4165 5323 50  0000 C CNN
+F 2 "" H 4150 5150 50  0001 C CNN
+F 3 "" H 4150 5150 50  0001 C CNN
+	1    4150 5150
+	1    0    0    -1
+$EndComp
+Text GLabel 4100 5450 0    50   Input ~ 0
 C2CK
 Text GLabel 4500 5550 0    50   Input ~ 0
@@
 Text GLabel 5900 3850 0    50   Input ~ 0
 LED
-Text GLabel 3650 4800 2    50   Input ~ 0
-LED
 Text GLabel 5700 5850 2    50   Input ~ 0
 LED
 Text GLabel 5700 6550 2    50   Input ~ 0
 A0
+$Comp
+L Connector_Generic:Conn_02x03_Odd_Even J2
+U 1 1 6127F01E
+P 5050 3500
+F 0 "J2" H 5100 3817 50  0000 C CNN
+F 1 "Tag-Connect" H 5100 3726 50  0000 C CNN
+F 2 "Connector:Tag-Connect_TC2030-IDC-NL_2x03_P1.27mm_Vertical" H 5050 3500 50  0001 C CNN
+F 3 "~" H 5050 3500 50  0001 C CNN
+	1    5050 3500
+	1    0    0    -1
+$EndComp
+$Comp
+L Device:R R6
+U 1 1 6128E69D
+P 4150 5300
+F 0 "R6" V 4250 5250 50  0000 L CNN
+F 1 "1k" V 4050 5250 50  0000 L CNN
+F 2 "Resistor_SMD:R_0603_1608Metric_Pad0.98x0.95mm_HandSolder" V 4080 5300 50  0001 C CNN
+F 3 "~" H 4150 5300 50  0001 C CNN
+	1    4150 5300
+	1    0    0    -1
+$EndComp
+Wire Wire Line
+	4500 5250 4300 5250
+Wire Wire Line
+	4300 5250 4300 5150
+Wire Wire Line
+	4300 5150 4150 5150
+Connection ~ 4150 5150
+Wire Wire Line
+	4500 5350 4300 5350
+Wire Wire Line
+	4300 5350 4300 5250
+Connection ~ 4300 5250
+Wire Wire Line
+	4100 5450 4150 5450
+Wire Wire Line
+	4500 5450 4150 5450
+Connection ~ 4150 5450
+Text GLabel 4850 3400 0    50   Input ~ 0
+BATT
+$Comp
+L power:+3.3V #PWR0105
+U 1 1 612F90A4
+P 9100 3400
+F 0 "#PWR0105" H 9100 3250 50  0001 C CNN
+F 1 "+3.3V" V 9150 3600 50  0000 C CNN
+F 2 "" H 9100 3400 50  0001 C CNN
+F 3 "" H 9100 3400 50  0001 C CNN
+	1    9100 3400
+	0    -1   -1   0
+$EndComp
+Wire Wire Line
+	9100 3400 9300 3400
+Wire Wire Line
+	9100 3500 9300 3500
 $EndSCHEMATC

Commit message: added high-voltage measurement
Parts:
- added R7: 110k, Resistor_SMD:R_0603_1608Metric_Pad0.98x0.95mm_HandSolder, symbol Device:R
- added R8: 10k, Resistor_SMD:R_0603_1608Metric_Pad0.98x0.95mm_HandSolder, symbol Device:R
Connections:
- net A3: now also R7.2, R8.1; no longer J1.6 (Pin_6)
- net GND: now also R8.2
- new net VHIGH: J1.6 (Pin_6), R7.1
Changed lines of the file:
@@
 $EndComp
 Text GLabel 9300 3300 0    50   Input ~ 0
-A3
+VHIGH
 Text GLabel 9300 3200 0    50   Input ~ 0
 A2
@@
 Wire Wire Line
 	9100 3500 9300 3500
+$Comp
+L Device:R R7
+U 1 1 6131256B
+P 7350 3200
+F 0 "R7" V 7450 3150 50  0000 L CNN
+F 1 "110k" V 7250 3150 50  0000 L CNN
+F 2 "Resistor_SMD:R_0603_1608Metric_Pad0.98x0.95mm_HandSolder" V 7280 3200 50  0001 C CNN
+F 3 "~" H 7350 3200 50  0001 C CNN
+	1    7350 3200
+	1    0    0    -1
+$EndComp
+$Comp
+L Device:R R8
+U 1 1 61316095
+P 7350 3600
+F 0 "R8" V 7450 3550 50  0000 L CNN
+F 1 "10k" V 7250 3550 50  0000 L CNN
+F 2 "Resistor_SMD:R_0603_1608Metric_Pad0.98x0.95mm_HandSolder" V 7280 3600 50  0001 C CNN
+F 3 "~" H 7350 3600 50  0001 C CNN
+	1    7350 3600
+	1    0    0    -1
+$EndComp
+$Comp
+L power:GND #PWR0110
+U 1 1 613169FE
+P 7350 3750
+F 0 "#PWR0110" H 7350 3500 50  0001 C CNN
+F 1 "GND" H 7355 3577 50  0000 C CNN
+F 2 "" H 7350 3750 50  0001 C CNN
+F 3 "" H 7350 3750 50  0001 C CNN
+	1    7350 3750
+	1    0    0    -1
+$EndComp
+Text GLabel 7350 3050 1    50   Input ~ 0
+VHIGH
+Wire Wire Line
+	7350 3350 7350 3450
+Text GLabel 7000 3450 0    50   Input ~ 0
+A3
+Wire Wire Line
+	7350 3450 7000 3450
+Connection ~ 7350 3450
 $EndSCHEMATC
