File: hardware/wireless_measurement_ard.sch (KiCad schematic (older format))
At the start: 27 parts, among them J1 Conn_01x08, J2 Tag-Connect, SW1 SW_SPDT, U1 EFM8LB1, U2 JDY-08, U3 MCP16415, U4 MAX9938, U5 MAX9938

Commit message: completed v1
Parts:
- removed H1, H2: MountingHole_Pad, MountingHole:MountingHole_2.2mm_M2_ISO7380_Pad, symbol Mechanical:MountingHole_Pad
- removed R2: 5R3, Resistor_SMD:R_0805_2012Metric_Pad1.15x1.40mm_HandSolder, symbol Device:R
- removed U4, U5: MAX9938, Package_TO_SOT_SMD:SOT-23-5_HandSoldering, symbol wireless_measurement_ard-rescue:MAX9938-gen_lib
- added U4: MAX44284, Package_TO_SOT_SMD:SOT-23-6_Handsoldering, symbol wireless_measurement_ard-rescue:MAX44284
- R1: value 5R3 -> 1R
Connections:
- net labels added: A4
- net labels removed: C2_IN, C2_OUT
- wire segments 68 -> 60
Changed lines of the file:
@@
-$EndComp
-$Comp
-L wireless_measurement_ard-rescue:MAX9938-gen_lib U4
-U 1 1 60F745CE
-P 8900 1750
-F 0 "U4" H 8900 2065 50  0000 C CNN
-F 1 "MAX9938" H 8900 1974 50  0000 C CNN
-F 2 "Package_TO_SOT_SMD:SOT-23-5_HandSoldering" H 8900 1450 50  0001 C CNN
-F 3 "http://www.farnell.com/datasheets/2345095.pdf" H 8900 1750 50  0001 C CNN
-	1    8900 1750
-	1    0    0    -1
-$EndComp
-$Comp
-L wireless_measurement_ard-rescue:MAX9938-gen_lib U5
-U 1 1 60F75707
-P 8900 2300
-F 0 "U5" H 8900 2615 50  0000 C CNN
-F 1 "MAX9938" H 8900 2524 50  0000 C CNN
-F 2 "Package_TO_SOT_SMD:SOT-23-5_HandSoldering" H 8900 2000 50  0001 C CNN
-F 3 "http://www.farnell.com/datasheets/2345095.pdf" H 8900 2300 50  0001 C CNN
-	1    8900 2300
-	1    0    0    -1
 $EndComp
 $Comp
@@
 	1    0    0    -1
 $EndComp
-$Comp
-L power:GND #PWR0102
-U 1 1 60F7644E
-P 8550 2400
-F 0 "#PWR0102" H 8550 2150 50  0001 C CNN
-F 1 "GND" H 8555 2227 50  0000 C CNN
-F 2 "" H 8550 2400 50  0001 C CNN
-F 3 "" H 8550 2400 50  0001 C CNN
-	1    8550 2400
-	1    0    0    -1
-$EndComp
-Wire Wire Line
-	8550 2200 8400 2200
 Wire Wire Line
 	8550 1650 8400 1650
-Text GLabel 8400 1650 0    50   Input ~ 0
+Text GLabel 9350 1450 2    50   Input ~ 0
 A0
-Text GLabel 8400 2200 0    50   Input ~ 0
+Text GLabel 9300 3000 0    50   Input ~ 0
 A1
 Wire Wire Line
@@
 Wire Wire Line
 	9350 1750 9350 1850
-Wire Wire Line
-	9250 2200 9250 2100
-Wire Wire Line
-	9250 2300 9250 2400
-Connection ~ 9450 2100
-Connection ~ 9450 2400
-Wire Wire Line
-	9450 2400 9650 2400
-Wire Wire Line
-	9250 2400 9450 2400
-Wire Wire Line
-	9450 2100 9650 2100
-Wire Wire Line
-	9250 2100 9450 2100
-$Comp
-L Device:R R2
-U 1 1 60F771F1
-P 9450 2250
-F 0 "R2" H 9520 2296 50  0000 L CNN
-F 1 "5R3" H 9520 2205 50  0000 L CNN
-F 2 "Resistor_SMD:R_0805_2012Metric_Pad1.15x1.40mm_HandSolder" V 9380 2250 50  0001 C CNN
-F 3 "~" H 9450 2250 50  0001 C CNN
-	1    9450 2250
-	1    0    0    -1
-$EndComp
 Connection ~ 9450 1550
 Connection ~ 9450 1850
@@
 P 9450 1700
 F 0 "R1" H 9520 1746 50  0000 L CNN
-F 1 "5R3" H 9520 1655 50  0000 L CNN
+F 1 "1R" H 9520 1655 50  0000 L CNN
 F 2 "Resistor_SMD:R_0805_2012Metric_Pad1.15x1.40mm_HandSolder" V 9380 1700 50  0001 C CNN
 F 3 "~" H 9450 1700 50  0001 C CNN
@@
 	1    0    0    -1
 $EndComp
-Wire Wire Line
-	9650 2100 9650 2200
-Wire Wire Line
-	9650 2300 9650 2400
 Wire Wire Line
 	9650 1850 9650 1750
@@
 	1    0    0    -1
 $EndComp
-Text GLabel 9300 3300 0    50   Input ~ 0
+Text GLabel 9300 3200 0    50   Input ~ 0
 VHIGH
-Text GLabel 9300 3200 0    50   Input ~ 0
+Text GLabel 9300 3100 0    50   Input ~ 0
 A2
 $Comp
@@
 	0    1    1    0
 $EndComp
+Text GLabel 9800 1750 2    50   Input ~ 0
+C1_IN
+Wire Wire Line
+	9650 1750 9800 1750
+Wire Wire Line
+	9650 1650 9800 1650
+Text GLabel 9300 2800 0    50   Input ~ 0
+C1_IN
 Text GLabel 9800 1650 2    50   Input ~ 0
-C1_IN
-Text GLabel 9800 2300 2    50   Input ~ 0
-C2_OUT
-Text GLabel 9800 2200 2    50   Input ~ 0
-C2_IN
-Wire Wire Line
-	9650 2200 9800 2200
-Wire Wire Line
-	9650 2300 9800 2300
-Wire Wire Line
-	9650 1750 9800 1750
-Wire Wire Line
-	9650 1650 9800 1650
+C1_OUT
 Text GLabel 9300 2900 0    50   Input ~ 0
-C1_IN
-Text GLabel 9800 1750 2    50   Input ~ 0
 C1_OUT
-Text GLabel 9300 2800 0    50   Input ~ 0
-C1_OUT
-Text GLabel 9300 3100 0    50   Input ~ 0
-C2_IN
-Text GLabel 9300 3000 0    50   Input ~ 0
-C2_OUT
 Text GLabel 8550 4250 0    50   Input ~ 0
 VIN
@@
 Wire Wire Line
 	8550 1750 8550 1850
-Connection ~ 8550 1850
-Wire Wire Line
-	8550 2300 8550 2400
-Connection ~ 8550 2400
 $Comp
 L power:+3.3V #PWR0118
@@
 Text GLabel 6200 4650 0    50   Input ~ 0
 VIN
-$Comp
-L Mechanical:MountingHole_Pad H1
-U 1 1 6108948B
-P 5550 2350
-F 0 "H1" H 5650 2399 50  0000 L CNN
-F 1 "MountingHole_Pad" H 5650 2308 50  0000 L CNN
-F 2 "MountingHole:MountingHole_2.2mm_M2_ISO7380_Pad" H 5550 2350 50  0001 C CNN
-F 3 "~" H 5550 2350 50  0001 C CNN
-	1    5550 2350
-	1    0    0    -1
-$EndComp
-$Comp
-L Mechanical:MountingHole_Pad H2
-U 1 1 61089F2F
-P 5900 2350
-F 0 "H2" H 6000 2399 50  0000 L CNN
-F 1 "MountingHole_Pad" H 6000 2308 50  0000 L CNN
-F 2 "MountingHole:MountingHole_2.2mm_M2_ISO7380_Pad" H 5900 2350 50  0001 C CNN
-F 3 "~" H 5900 2350 50  0001 C CNN
-	1    5900 2350
-	1    0    0    -1
-$EndComp
 $Comp
 L MCU_SiliconLabs:EFM8LB1 U1
@@
 	7350 3450 7000 3450
 Connection ~ 7350 3450
+$Comp
+L wireless_measurement_ard-rescue:MAX44284 U4
+U 1 1 612DBC77
+P 8900 1650
+F 0 "U4" H 8900 1975 50  0000 C CNN
+F 1 "MAX44284" H 8900 1884 50  0000 C CNN
+F 2 "Package_TO_SOT_SMD:SOT-23-6_Handsoldering" H 8900 1450 50  0001 C CNN
+F 3 "https://datasheets.maximintegrated.com/en/ds/MAX44284.pdf" H 8900 1450 50  0001 C CNN
+	1    8900 1650
+	1    0    0    -1
+$EndComp
+Wire Wire Line
+	9250 1550 9250 1450
+Wire Wire Line
+	9250 1450 9350 1450
+Wire Wire Line
+	8550 1550 8400 1550
+Wire Wire Line
+	8400 1550 8400 1650
+$Comp
+L power:+3.3V #PWR0111
+U 1 1 612E1F0B
+P 8400 1550
+F 0 "#PWR0111" H 8400 1400 50  0001 C CNN
+F 1 "+3.3V" H 8415 1723 50  0000 C CNN
+F 2 "" H 8400 1550 50  0001 C CNN
+F 3 "" H 8400 1550 50  0001 C CNN
+	1    8400 1550
+	1    0    0    -1
+$EndComp
+Connection ~ 8400 1550
+Text GLabel 5700 5750 2    50   Input ~ 0
+A4
+Text GLabel 9300 3300 0    50   Input ~ 0
+A4
 $EndSCHEMATC

Commit message: mini version
Other:
- moved on the sheet: C5, C6, D1, R3, R6, SW1, U1

Commit message: updated board
Parts:
- removed Battery1: Conn_01x02, Connector_PinSocket_2.54mm:PinSocket_1x02_P2.54mm_Vertical, symbol Connector_Generic:Conn_01x02
- removed J2: Tag-Connect, Connector:Tag-Connect_TC2030-IDC-NL_2x03_P1.27mm_Vertical, symbol Connector_Generic:Conn_02x03_Odd_Even
- added C7: 4.7uF, Capacitor_SMD:C_0603_1608Metric_Pad1.08x0.95mm_HandSolder, symbol Device:C
- J1: footprint Connector_PinHeader_2.54mm:PinHeader_1x08_P2.54mm_Horizontal -> Connector_PinHeader_2.54mm:PinHeader_2x04_P2.54mm_Vertical
- R3: footprint Resistor_SMD:R_0603_1608Metric_Pad1.05x0.95mm_HandSolder -> Resistor_SMD:R_0603_1608Metric_Pad0.98x0.95mm_HandSolder
Connections:
- wire segments 60 -> 59
Changed lines of the file:
@@
 F 0 "J1" H 9580 3092 50  0000 L CNN
 F 1 "Conn_01x08" H 9580 3001 50  0000 L CNN
-F 2 "Connector_PinHeader_2.54mm:PinHeader_1x08_P2.54mm_Horizontal" H 9500 3100 50  0001 C CNN
+F 2 "Connector_PinHeader_2.54mm:PinHeader_2x04_P2.54mm_Vertical" H 9500 3100 50  0001 C CNN
 F 3 "~" H 9500 3100 50  0001 C CNN
 	1    9500 3100
 	1    0    0    -1
 $EndComp
-Text GLabel 9300 3200 0    50   Input ~ 0
+Text GLabel 9300 3100 0    50   Input ~ 0
 VHIGH
-Text GLabel 9300 3100 0    50   Input ~ 0
+Text GLabel 8300 2700 0    50   Input ~ 0
 A2
 $Comp
@@
 Wire Wire Line
 	8700 5000 8850 5000
-Text GLabel 10250 2800 0    50   Input ~ 0
-BATT
-$Comp
-L Connector_Generic:Conn_01x02 Battery1
-U 1 1 60FE7457
-P 10450 2800
-F 0 "Battery1" H 10530 2792 50  0000 L CNN
-F 1 "Conn_01x02" H 10530 2701 50  0000 L CNN
-F 2 "Connector_PinSocket_2.54mm:PinSocket_1x02_P2.54mm_Vertical" H 10450 2800 50  0001 C CNN
-F 3 "~" H 10450 2800 50  0001 C CNN
-	1    10450 2800
-	1    0    0    -1
-$EndComp
-$Comp
-L power:GND #PWR0117
-U 1 1 60FE7F19
-P 10250 2900
-F 0 "#PWR0117" H 10250 2650 50  0001 C CNN
-F 1 "GND" H 10255 2727 50  0000 C CNN
-F 2 "" H 10250 2900 50  0001 C CNN
-F 3 "" H 10250 2900 50  0001 C CNN
-	1    10250 2900
-	1    0    0    -1
-$EndComp
 Wire Wire Line
 	8550 1750 8550 1850
@@
 STATUS
 Connection ~ 4850 4650
-$Comp
-L power:GND #PWR0121
-U 1 1 610243BD
-P 3400 3900
-F 0 "#PWR0121" H 3400 3650 50  0001 C CNN
-F 1 "GND" H 3405 3727 50  0000 C CNN
-F 2 "" H 3400 3900 50  0001 C CNN
-F 3 "" H 3400 3900 50  0001 C CNN
-	1    3400 3900
-	1    0    0    -1
-$EndComp
-Text GLabel 2900 3900 0    50   Input ~ 0
-C2D
-Text GLabel 2900 3800 0    50   Input ~ 0
-C2CK
 Wire Wire Line
 	8550 4450 8950 4450
@@
 F 0 "R3" V 6400 4750 50  0000 L CNN
 F 1 "1k" V 6200 4750 50  0000 L CNN
-F 2 "Resistor_SMD:R_0603_1608Metric_Pad1.05x0.95mm_HandSolder" V 6230 4800 50  0001 C CNN
+F 2 "Resistor_SMD:R_0603_1608Metric_Pad0.98x0.95mm_HandSolder" V 6230 4800 50  0001 C CNN
 F 3 "~" H 6300 4800 50  0001 C CNN
 	1    6300 4800
@@
 A0
 $Comp
-L Connector_Generic:Conn_02x03_Odd_Even J2
-U 1 1 6127F01E
-P 3100 3800
-F 0 "J2" H 3150 4117 50  0000 C CNN
-F 1 "Tag-Connect" H 3150 4026 50  0000 C CNN
-F 2 "Connector:Tag-Connect_TC2030-IDC-NL_2x03_P1.27mm_Vertical" H 3100 3800 50  0001 C CNN
-F 3 "~" H 3100 3800 50  0001 C CNN
-	1    3100 3800
-	1    0    0    -1
-$EndComp
-$Comp
 L Device:R R6
 U 1 1 6128E69D
@@
 	5250 1550 4900 1550
 Connection ~ 4900 1550
-Text GLabel 2900 3700 0    50   Input ~ 0
-BATT
-$Comp
-L power:+3.3V #PWR0105
-U 1 1 612F90A4
-P 9100 3400
-F 0 "#PWR0105" H 9100 3250 50  0001 C CNN
-F 1 "+3.3V" V 9150 3600 50  0000 C CNN
-F 2 "" H 9100 3400 50  0001 C CNN
-F 3 "" H 9100 3400 50  0001 C CNN
-	1    9100 3400
-	0    -1   -1   0
-$EndComp
-Wire Wire Line
-	9100 3400 9300 3400
 Wire Wire Line
 	9100 3500 9300 3500
@@
 Text GLabel 6450 1850 2    50   Input ~ 0
 A4
+Text GLabel 9300 3400 0    50   Input ~ 0
+BATT
+Text GLabel 9300 3200 0    50   Input ~ 0
+C2CK
 Text GLabel 9300 3300 0    50   Input ~ 0
-A4
+C2D
+$Comp
+L Device:C C7
+U 1 1 613D1737
+P 5250 1100
+F 0 "C7" H 5000 1150 50  0000 L CNN
+F 1 "4.7uF" H 4950 1050 50  0000 L CNN
+F 2 "Capacitor_SMD:C_0603_1608Metric_Pad1.08x0.95mm_HandSolder" H 5288 950 50  0001 C CNN
+F 3 "~" H 5250 1100 50  0001 C CNN
+	1    5250 1100
+	1    0    0    -1
+$EndComp
+$Comp
+L power:GND #PWR0102
+U 1 1 613D2357
+P 5250 950
+F 0 "#PWR0102" H 5250 700 50  0001 C CNN
+F 1 "GND" H 5255 777 50  0000 C CNN
+F 2 "" H 5250 950 50  0001 C CNN
+F 3 "" H 5250 950 50  0001 C CNN
+	1    5250 950
+	0    -1   -1   0
+$EndComp
 $EndSCHEMATC

Commit message: update to nano version
Parts:
- SW1: footprint Button_Switch_SMD:SW_SPDT_CK-JS102011SAQN -> ben_common:SW_SPDT_CK-JS102011SAQN
- U1: symbol MCU_SiliconLabs:EFM8LB1 -> wireless_measurement_ard-rescue:EFM8LB1-MCU_SiliconLabs
- U2: footprint JDY-08:JDY-08_HandSoldering -> ben_common:JDY-08_HandSoldering
Changed lines of the file:
@@
 F 0 "U2" H 3150 3187 60  0000 C CNN
 F 1 "JDY-08" H 3150 3081 60  0000 C CNN
-F 2 "JDY-08:JDY-08_HandSoldering" H 5000 2000 60  0001 C CNN
+F 2 "ben_common:JDY-08_HandSoldering" H 5000 2000 60  0001 C CNN
 F 3 "https://github.com/kichMan/JDY-08" H 5000 2000 60  0001 C CNN
 	1    3150 2100
@@
 F 0 "SW1" H 10500 3735 50  0000 C CNN
 F 1 "SW_SPDT" H 10500 3644 50  0000 C CNN
-F 2 "Button_Switch_SMD:SW_SPDT_CK-JS102011SAQN" H 10500 3450 50  0001 C CNN
+F 2 "ben_common:SW_SPDT_CK-JS102011SAQN" H 10500 3450 50  0001 C CNN
 F 3 "~" H 10500 3450 50  0001 C CNN
 	1    10500 3450
@@
 VIN
 $Comp
-L MCU_SiliconLabs:EFM8LB1 U1
+L wireless_measurement_ard-rescue:EFM8LB1-MCU_SiliconLabs U1
 U 1 1 611E9E7B
 P 5850 2000

Commit message: Added new code for mini
Parts:
- added C8: 0.1uF, Capacitor_SMD:C_0603_1608Metric_Pad1.08x0.95mm_HandSolder, symbol Device:C
- added R2: 10k, Resistor_SMD:R_0603_1608Metric_Pad0.98x0.95mm_HandSolder, symbol Device:R
- added U5: DRV5021, Package_TO_SOT_SMD:SOT-23, symbol ben_common:DRV5021
- U1: symbol wireless_measurement_ard-rescue:EFM8LB1-MCU_SiliconLabs -> wireless_measurement_ard-rescue:EFM8LB1-MCU_SiliconLabs-wireless_measurement_ard-rescue
Connections:
- net +3V3: now also C8.1, R2.1, U5.1 (VCC)
- net GND: now also C8.2, U5.3 (GND)
- net HALL_PIN: now reaches U1.30 (P0.3)
- net HALL_PIN: now also R2.2, U5.2 (OUT)
Changed lines of the file:
@@
 Text GLabel 9300 3100 0    50   Input ~ 0
 VHIGH
-Text GLabel 8300 2700 0    50   Input ~ 0
-A2
 $Comp
 L power:GND #PWR0106
@@
 VIN
 $Comp
-L wireless_measurement_ard-rescue:EFM8LB1-MCU_SiliconLabs U1
+L wireless_measurement_ard-rescue:EFM8LB1-MCU_SiliconLabs-wireless_measurement_ard-rescue U1
 U 1 1 611E9E7B
 P 5850 2000
@@
 	0    -1   -1   0
 $EndComp
+Text GLabel 6450 1450 2    50   Input ~ 0
+HALL_PIN
+$Comp
+L ben_common:DRV5021 U5
+U 1 1 6148F942
+P 7400 1750
+F 0 "U5" H 7400 2025 50  0000 C CNN
+F 1 "DRV5021" H 7400 1950 50  0000 C CNN
+F 2 "Package_TO_SOT_SMD:SOT-23" H 7100 1950 50  0001 C CNN
+F 3 "" H 7100 1950 50  0001 C CNN
+	1    7400 1750
+	1    0    0    -1
+$EndComp
+$Comp
+L power:GND #PWR0105
+U 1 1 6149026D
+P 7700 2100
+F 0 "#PWR0105" H 7700 1850 50  0001 C CNN
+F 1 "GND" H 7705 1927 50  0000 C CNN
+F 2 "" H 7700 2100 50  0001 C CNN
+F 3 "" H 7700 2100 50  0001 C CNN
+	1    7700 2100
+	1    0    0    -1
+$EndComp
+$Comp
+L power:+3.3V #PWR0117
+U 1 1 61490741
+P 7100 1750
+F 0 "#PWR0117" H 7100 1600 50  0001 C CNN
+F 1 "+3.3V" H 7115 1923 50  0000 C CNN
+F 2 "" H 7100 1750 50  0001 C CNN
+F 3 "" H 7100 1750 50  0001 C CNN
+	1    7100 1750
+	1    0    0    -1
+$EndComp
+$Comp
+L power:+3.3V #PWR0120
+U 1 1 61490CF5
+P 7800 1400
+F 0 "#PWR0120" H 7800 1250 50  0001 C CNN
+F 1 "+3.3V" H 7815 1573 50  0000 C CNN
+F 2 "" H 7800 1400 50  0001 C CNN
+F 3 "" H 7800 1400 50  0001 C CNN
+	1    7800 1400
+	1    0    0    -1
+$EndComp
+$Comp
+L Device:R R2
+U 1 1 614912CF
+P 7800 1550
+F 0 "R2" H 7870 1596 50  0000 L CNN
+F 1 "10k" H 7870 1505 50  0000 L CNN
+F 2 "Resistor_SMD:R_0603_1608Metric_Pad0.98x0.95mm_HandSolder" V 7730 1550 50  0001 C CNN
+F 3 "~" H 7800 1550 50  0001 C CNN
+	1    7800 1550
+	1    0    0    -1
+$EndComp
+Wire Wire Line
+	7700 1700 7800 1700
+Text GLabel 8000 1700 2    50   Input ~ 0
+HALL_PIN
+Wire Wire Line
+	7800 1700 8000 1700
+Connection ~ 7800 1700
+$Comp
+L Device:C C8
+U 1 1 6149AFDF
+P 7100 1900
+F 0 "C8" H 6850 1950 50  0000 L CNN
+F 1 "0.1uF" H 6800 1850 50  0000 L CNN
+F 2 "Capacitor_SMD:C_0603_1608Metric_Pad1.08x0.95mm_HandSolder" H 7138 1750 50  0001 C CNN
+F 3 "~" H 7100 1900 50  0001 C CNN
+	1    7100 1900
+	1    0    0    -1
+$EndComp
+Connection ~ 7100 1750
+Wire Wire Line
+	7100 2050 7700 2050
+Wire Wire Line
+	7700 2050 7700 2100
+Wire Wire Line
+	7700 1850 7700 2050
+Connection ~ 7700 2050
 $EndSCHEMATC
