File: hardware/_autosave-wireless_measurement_ard.kicad_pcb (KiCad board)
At the start: 2 copper layers, 30 x 23 mm, 23 parts, among them J1 Conn_01x08, J2 Tag-Connect, SW1 SW_SPDT, U1 EFM8LB1, U2 JDY-08, U3 MCP16415, U4 MAX44284

Commit message: fixed powersupply
Parts:
- added C7: 4.7uF, Capacitor_SMD:C_0603_1608Metric_Pad1.08x0.95mm_HandSolder, B.Cu at (126.3, 84.3)
Routing:
- net GND: track 59.3 -> 73.2 mm
- net Net-(C7-Pad2): track 0.00 -> 3.55 mm
- net +3V3: track 77.0 -> 78.7 mm
- net ARD_TX: track 10.7 -> 9.26 mm
- net ARD_RX: track 11.7 -> 12.7 mm
- net A4: track 18.5 -> 19.1 mm
Other:
- board text added: "OFF"
- board text added: "ON"
- board text added: "SWM-mini-2 Sep 21"
- board text removed: "SWM-mini Sep 21"
